File: glitcher/glitcher/glitcher.kicad_sch (KiCad schematic)
At the start: 3 parts, among them J1 Barrel_Jack, U1 SC0915, U2 CMOD_A7

Commit message: save
Parts:
- added D7: D_Schottky, symbol Device:D_Schottky
Connections:
- net VCC: now also D7.1 (K); no longer U2.24 (VU)
- new net: D7.2 (A), U2.24 (VU)
Changed lines of the file:
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@@
     (stroke (width 0) (type default) (color 0 0 0 0))
   )
-  (wire (pts (xy 146.05 140.97) (xy 154.94 140.97))
+  (wire (pts (xy 144.78 154.94) (xy 154.94 154.94))
+    (stroke (width 0) (type default) (color 0 0 0 0))
+  )
+  (wire (pts (xy 137.16 154.94) (xy 129.54 154.94))
     (stroke (width 0) (type default) (color 0 0 0 0))
   )
@@
     (stroke (width 0) (type default) (color 0 0 0 0))
   )
+  (wire (pts (xy 129.54 156.21) (xy 125.73 156.21))
+    (stroke (width 0) (type default) (color 0 0 0 0))
+  )
   (wire (pts (xy 24.13 82.55) (xy 35.56 82.55))
     (stroke (width 0) (type default) (color 0 0 0 0))
@@
     (stroke (width 0) (type default) (color 0 0 0 0))
   )
+  (wire (pts (xy 154.94 154.94) (xy 154.94 140.97))
+    (stroke (width 0) (type default) (color 0 0 0 0))
+  )
   (wire (pts (xy 121.92 115.57) (xy 133.35 115.57))
     (stroke (width 0) (type default) (color 0 0 0 0))
@@
   )
   (wire (pts (xy 24.13 120.65) (xy 35.56 120.65))
+    (stroke (width 0) (type default) (color 0 0 0 0))
+  )
+  (wire (pts (xy 129.54 154.94) (xy 129.54 156.21))
     (stroke (width 0) (type default) (color 0 0 0 0))
   )
@@
     )
     (pin "1")
+  )
+  (symbol (lib_id "Device:D_Schottky") (at 140.97 154.94 0) (unit 1)
+    (in_bom yes) (on_board yes) (fields_autoplaced)
+    (property "Reference" "D7" (id 0) (at 140.6525 148.59 0))
+    (property "Value" "D_Schottky" (id 1) (at 140.6525 151.13 0))
+    (property "Footprint" "" (id 2) (at 140.97 154.94 0)
+      (effects (font (size 1.27 1.27)) hide)
+    )
+    (property "Datasheet" "~" (id 3) (at 140.97 154.94 0)
+      (effects (font (size 1.27 1.27)) hide)
+    )
+    (pin "1")
+    (pin "2")
   )
   (symbol (lib_id "Connector:Barrel_Jack") (at 31.75 31.75 0) (unit 1)
@@
     (pin "1")
   )
-  (symbol (lib_id "power:VCC") (at 146.05 140.97 0) (unit 1)
-    (in_bom yes) (on_board yes) (fields_autoplaced)
-    (property "Reference" "#PWR0112" (id 0) (at 146.05 144.78 0)
-      (effects (font (size 1.27 1.27)) hide)
-    )
-    (property "Value" "VCC" (id 1) (at 146.05 135.89 0))
-    (property "Footprint" "" (id 2) (at 146.05 140.97 0)
-      (effects (font (size 1.27 1.27)) hide)
-    )
-    (property "Datasheet" "" (id 3) (at 146.05 140.97 0)
+  (symbol (lib_id "power:VCC") (at 125.73 156.21 0) (unit 1)
+    (in_bom yes) (on_board yes) (fields_autoplaced)
+    (property "Reference" "#PWR0112" (id 0) (at 125.73 160.02 0)
+      (effects (font (size 1.27 1.27)) hide)
+    )
+    (property "Value" "VCC" (id 1) (at 125.73 151.13 0))
+    (property "Footprint" "" (id 2) (at 125.73 156.21 0)
+      (effects (font (size 1.27 1.27)) hide)
+    )
+    (property "Datasheet" "" (id 3) (at 125.73 156.21 0)
       (effects (font (size 1.27 1.27)) hide)
     )
@@
       (reference "D6") (unit 1) (value "LED") (footprint "LED_SMD:LED_0603_1608Metric_Pad1.05x0.95mm_HandSolder")
     )
+    (path "/30b6f105-b8ee-4acc-bcdb-369e9c021283"
+      (reference "D7") (unit 1) (value "D_Schottky") (footprint "Diode_SMD:D_SOD-123F")
+    )
     (path "/b472a744-f1dd-43ec-9020-370e486042ce/10febe5f-8747-4f68-aeef-060e8a91ecdf"
       (reference "HS2_OUT1") (unit 1) (value "Conn_Coaxial") (footprint "Connector_Coaxial:SMA_Molex_73251-2120_EdgeMount_Horizontal")
@@
       (reference "J7") (unit 1) (value "Conn_01x03") (footprint "Connector_PinHeader_2.54mm:PinHeader_1x03_P2.54mm_Vertical")
     )
+    (path "/b472a744-f1dd-43ec-9020-370e486042ce/8fd3448a-2c13-451e-8b1b-bad8e3e9f797"
+      (reference "J_LEFTEXP1") (unit 1) (value "Conn_01x20") (footprint "Connector_PinHeader_2.54mm:PinHeader_1x20_P2.54mm_Vertical")
+    )
+    (path "/b472a744-f1dd-43ec-9020-370e486042ce/a2e2d058-d14f-4a05-a53b-27dfbc867df8"
+      (reference "J_LEFTEXP_OUTER1") (unit 1) (value "Conn_01x20") (footprint "Connector_PinHeader_2.54mm:PinHeader_1x20_P2.54mm_Vertical")
+    )
+    (path "/b472a744-f1dd-43ec-9020-370e486042ce/c9ccd606-4d54-4cb4-bcad-a110124d5c1e"
+      (reference "J_RIGHTEXP1") (unit 1) (value "Conn_01x20") (footprint "Connector_PinHeader_2.54mm:PinHeader_1x20_P2.54mm_Vertical")
+    )
+    (path "/b472a744-f1dd-43ec-9020-370e486042ce/f5b31508-212f-453f-b286-cc65f9e07b18"
+      (reference "J_RIGHTEXP_OUTER1") (unit 1) (value "Conn_01x20") (footprint "Connector_PinHeader_2.54mm:PinHeader_1x20_P2.54mm_Vertical")
+    )
     (path "/b472a744-f1dd-43ec-9020-370e486042ce/09d79d6c-44ce-4338-95f2-29a1cf801993"

Commit message: lolsave
Parts:
- D7: footprint (none) -> Diode_SMD:D_SOD-123F
Connections:
- net RPI_GP0: now reaches U1.1 (UART0_TX/I2C0_SDA/SPI0_RX/GP0)
- net RPI_GP0: now also U2.26 (PIO26)
- net RPI_GP7: now reaches U1.10 (I2C1_SCL/SPI0_TX/GP7)
- net RPI_GP8: now reaches U1.11 (UART1_TX/I2C0_SDA/SPI1_RX/GP8)
- net RPI_GP9: now reaches U1.12 (UART1_RX/I2C0_SCL/SPI1_CSn/GP9)
- net RPI_GP10: now reaches U1.14 (I2C1_SDA/SPI1_SCK/GP10)
- net RPI_GP11: now reaches U1.15 (I2C1_SCL/SPI1_TX/GP11)
- net RPI_GP12: now reaches U1.16 (UART0_TX/I2C0_SDA/GPI1_RX/GP12)
- net RPI_GP13: now reaches U1.17 (UART0_RX/I2C0_SCL/SPI1_CSn/GP13)
- net RPI_GP14: now reaches U1.19 (I2C1_SDA/SPI1_SCK/GP14)
- net RPI_GP1: now reaches U1.2 (UART0_RX/I2C0_SCL/GPI0_CSn/GP1)
- net RPI_GP1: now also U2.27 (PIO27)
- net RPI_GP15: now reaches U1.20 (I2C1_SCL/SPI1_TX/GP15)
- net RPI_GP16: now reaches U1.21 (UART0_TX/I2C0_SDA/SPI0_RX/GP16)
- net RPI_GP17: now reaches U1.22 (UART0_RX/I2C0_SCL/SPI0_CSn/GP17)
- net RPI_GP2: now reaches U1.4 (I2C1_SDA/SPI0_SCK/GP2)
- net RPI_GP3: now reaches U1.5 (I2C1_SCL/SPI0_TX/GP3)
- net RPI_GP4: now reaches U1.6 (UART1_TX/I2C0_SDA/SPI0_RX/GP4)
- net RPI_GP5: now reaches U1.7 (UART1_RX/I2C0_SCL/SPI0_CSn/GP5)
- net RPI_GP6: now reaches U1.9 (I2C1_SDA/SPI0_SCK/GP6)
- net MAX4619_C: now reaches U2.1 (PIO01)
- net FPGA_GPIO_6: now reaches U2.10 (PIO10)
- net FPGA_GPIO_5: now reaches U2.11 (PIO11)
- net FPGA_GPIO_4: now reaches U2.12 (PIO12)
- net FPGA_GPIO_3: now reaches U2.13 (PIO13)
- net FPGA_GPIO_2: now reaches U2.14 (PIO14)
- net FPGA_GPIO_1: now reaches U2.15 (PIO15)
- net MAX4619_B: now reaches U2.2 (PIO02)
- net MAX4619_A: now reaches U2.3 (PIO03)
- net FPGA_GPIO_12: now reaches U2.4 (PIO04)
- net FPGA_GPIO_11: now reaches U2.5 (PIO05)
- net FPGA_GPIO_10: now reaches U2.6 (PIO06)
- net FPGA_GPIO_9: now reaches U2.7 (PIO07)
- net FPGA_GPIO_8: now reaches U2.8 (PIO08)
- net FPGA_GPIO_7: now reaches U2.9 (PIO09)
Other:
- added sheet shield_connector (shield_connector.kicad_sch)
- moved on the sheet: D7, U2

Commit message: save
Parts:
- removed D7: D_Schottky, Diode_SMD:D_SOD-123F, symbol Device:D_Schottky
- added JP2, JP3: SolderJumper_2_Open, Jumper:SolderJumper-2_P1.3mm_Open_Pad1.0x1.5mm, symbol Jumper:SolderJumper_2_Open
Connections:
- net VCC: now also JP2.2 (B), JP3.1 (A); no longer U1.39 (VSYS)
- net at U2.24 (VU): now also JP3.2 (B)
- new net: JP2.1 (A), U1.39 (VSYS)

Commit message: prod1
Parts:
- added FB1: FerriteBead, Inductor_SMD:L_0805_2012Metric_Pad1.05x1.20mm_HandSolder, symbol Device:FerriteBead
- added TP1, TP2: TestPoint, TestPoint:TestPoint_Pad_D3.0mm, symbol Connector:TestPoint
- U1: footprint DIP-40_W15.24mm_Socket_LongPads -> all_lib:rpi_socket_fixed
Connections:
- net VCC: now also FB1.1
- net FPGA_4: now reaches U1.27 (I2C0_SCL/GP21)
- net FPGA_4: now also U2.29 (PIO29)
- net FPGA_3: now reaches U1.29 (GP22)
- net FPGA_3: now also U2.28 (PIO28)
- net at U1.31 (I2C1_SDA/ADC0/GP26): now also TP2.1
- net at U1.32 (I2C1_SCL/ADC1/GP27): now also TP1.1
- net at JP3.2 (B), U2.24 (VU): now also FB1.2
Other:
- note added: "width between sides should be 700mils double check pcbnew do not use dip40"
Changed lines of the file:
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@@
 (kicad_sch (version 20211123) (generator eeschema)
   (paper "A4")
+  (junction (at 156.21 156.21) (diameter 0) (color 0 0 0 0)
+  )
+  (junction (at 179.07 156.21) (diameter 0) (color 0 0 0 0)
+  )
   (no_connect (at 86.36 95.25))
   (no_connect (at 67.31 76.2))
@@
     (stroke (width 0) (type default) (color 0 0 0 0))
   )
+  (wire (pts (xy 172.72 144.78) (xy 179.07 144.78))
+    (stroke (width 0) (type default) (color 0 0 0 0))
+  )
+  (wire (pts (xy 179.07 156.21) (xy 189.23 156.21))
+    (stroke (width 0) (type default) (color 0 0 0 0))
+  )
   (wire (pts (xy 30.48 128.27) (xy 35.56 128.27))
     (stroke (width 0) (type default) (color 0 0 0 0))
@@
     (stroke (width 0) (type default) (color 0 0 0 0))
   )
-  (wire (pts (xy 171.45 156.21) (xy 189.23 156.21))
+  (wire (pts (xy 171.45 156.21) (xy 179.07 156.21))
+    (stroke (width 0) (type default) (color 0 0 0 0))
+  )
+  (wire (pts (xy 217.17 132.08) (xy 223.52 132.08))
     (stroke (width 0) (type default) (color 0 0 0 0))
   )
@@
     (stroke (width 0) (type default) (color 0 0 0 0))
   )
+  (wire (pts (xy 217.17 134.62) (xy 223.52 134.62))
+    (stroke (width 0) (type default) (color 0 0 0 0))
+  )
   (wire (pts (xy 30.48 87.63) (xy 35.56 87.63))
     (stroke (width 0) (type default) (color 0 0 0 0))
@@
     (stroke (width 0) (type default) (color 0 0 0 0))
   )
+  (wire (pts (xy 121.92 138.43) (xy 124.46 138.43))
+    (stroke (width 0) (type default) (color 0 0 0 0))
+  )
   (wire (pts (xy 24.13 82.55) (xy 35.56 82.55))
     (stroke (width 0) (type default) (color 0 0 0 0))
@@
     (stroke (width 0) (type default) (color 0 0 0 0))
   )
+  (wire (pts (xy 121.92 130.81) (xy 142.24 130.81))
+    (stroke (width 0) (type default) (color 0 0 0 0))
+  )
   (wire (pts (xy 189.23 156.21) (xy 189.23 142.24))
     (stroke (width 0) (type default) (color 0 0 0 0))
@@
     (stroke (width 0) (type default) (color 0 0 0 0))
   )
+  (wire (pts (xy 156.21 144.78) (xy 165.1 144.78))
+    (stroke (width 0) (type default) (color 0 0 0 0))
+  )
   (wire (pts (xy 39.37 34.29) (xy 44.45 34.29))
     (stroke (width 0) (type default) (color 0 0 0 0))
@@
     (stroke (width 0) (type default) (color 0 0 0 0))
   )
+  (wire (pts (xy 121.92 143.51) (xy 124.46 143.51))
+    (stroke (width 0) (type default) (color 0 0 0 0))
+  )
   (wire (pts (xy 24.13 120.65) (xy 35.56 120.65))
     (stroke (width 0) (type default) (color 0 0 0 0))
@@
     (stroke (width 0) (type default) (color 0 0 0 0))
   )
+  (wire (pts (xy 121.92 133.35) (xy 142.24 133.35))
+    (stroke (width 0) (type default) (color 0 0 0 0))
+  )
   (wire (pts (xy 184.15 114.3) (xy 189.23 114.3))
     (stroke (width 0) (type default) (color 0 0 0 0))
@@
     (stroke (width 0) (type default) (color 0 0 0 0))
   )
+  (wire (pts (xy 156.21 156.21) (xy 156.21 144.78))
+    (stroke (width 0) (type default) (color 0 0 0 0))
+  )
   (wire (pts (xy 189.23 101.6) (xy 184.15 101.6))
     (stroke (width 0) (type default) (color 0 0 0 0))
@@
     (stroke (width 0) (type default) (color 0 0 0 0))
   )
+  (wire (pts (xy 179.07 144.78) (xy 179.07 156.21))
+    (stroke (width 0) (type default) (color 0 0 0 0))
+  )
   (wire (pts (xy 30.48 77.47) (xy 35.56 77.47))
     (stroke (width 0) (type default) (color 0 0 0 0))
@@
     (stroke (width 0) (type default) (color 0 0 0 0))
   )
-  (wire (pts (xy 149.86 156.21) (xy 157.48 156.21))
+  (wire (pts (xy 149.86 156.21) (xy 156.21 156.21))
+    (stroke (width 0) (type default) (color 0 0 0 0))
+  )
+  (wire (pts (xy 156.21 156.21) (xy 157.48 156.21))
     (stroke (width 0) (type default) (color 0 0 0 0))
   )
@@
     (stroke (width 0) (type default) (color 0 0 0 0))
   )
+  (text "width between sides should be 700mils\ndouble check pcbnew do not use dip40"
+    (at 59.69 60.96 0)
+    (effects (font (size 1.27 1.27)) (justify left bottom))
+  )
   (global_label "RPI_GP1" (shape input) (at 30.48 80.01 180) (fields_autoplaced)
     (effects (font (size 1.27 1.27)) (justify right))
     (property "Intersheet References" "${INTERSHEET_REFS}" (id 0) (at 20.205 79.9306 0)
       (effects (font (size 1.27 1.27)) (justify right) hide)
+    )
+  )
+  (global_label "FPGA_3" (shape input) (at 124.46 138.43 0) (fields_autoplaced)
+    (effects (font (size 1.27 1.27)) (justify left))
+    (property "Intersheet References" "${INTERSHEET_REFS}" (id 0) (at 133.7674 138.3506 0)
+      (effects (font (size 1.27 1.27)) (justify left) hide)
     )
   )
@@
     )
   )
+  (global_label "FPGA_3" (shape input) (at 223.52 134.62 0) (fields_autoplaced)
+    (effects (font (size 1.27 1.27)) (justify left))
+    (property "Intersheet References" "${INTERSHEET_REFS}" (id 0) (at 232.8274 134.5406 0)
+      (effects (font (size 1.27 1.27)) (justify left) hide)
+    )
+  )
   (global_label "RPI_GP5" (shape input) (at 30.48 92.71 180) (fields_autoplaced)
     (effects (font (size 1.27 1.27)) (justify right))
@@
     (property "Intersheet References" "${INTERSHEET_REFS}" (id 0) (at 169.3998 104.2194 0)
       (effects (font (size 1.27 1.27)) (justify right) hide)
+    )
+  )
+  (global_label "FPGA_4" (shape input) (at 124.46 143.51 0) (fields_autoplaced)
+    (effects (font (size 1.27 1.27)) (justify left))
+    (property "Intersheet References" "${INTERSHEET_REFS}" (id 0) (at 133.7674 143.4306 0)
+      (effects (font (size 1.27 1.27)) (justify left) hide)
+    )
+  )
+  (global_label "FPGA_4" (shape input) (at 223.52 132.08 0) (fields_autoplaced)
+    (effects (font (size 1.27 1.27)) (justify left))
+    (property "Intersheet References" "${INTERSHEET_REFS}" (id 0) (at 232.8274 132.0006 0)
+      (effects (font (size 1.27 1.27)) (justify left) hide)
     )
   )
@@
       (effects (font (size 1.524 1.524)))
     )
-    (property "Footprint" "DIP-40_W15.24mm_Socket_LongPads" (id 2) (at 81.28 68.834 0)
+    (property "Footprint" "all_lib:rpi_socket_fixed" (id 2) (at 81.28 68.834 0)
       (effects (font (size 1.524 1.524)) hide)
     )
@@
     (pin "9")
   )
+  (symbol (lib_id "Connector:TestPoint") (at 142.24 130.81 270) (unit 1)
+    (in_bom yes) (on_board yes) (fields_autoplaced)
+    (property "Reference" "TP1" (id 0) (at 147.32 129.5399 90)
+      (effects (font (size 1.27 1.27)) (justify left))
+    )
+    (property "Value" "TestPoint" (id 1) (at 147.32 132.0799 90)
+      (effects (font (size 1.27 1.27)) (justify left))
+    )
+    (property "Footprint" "TestPoint:TestPoint_Pad_D3.0mm" (id 2) (at 142.24 135.89 0)
+      (effects (font (size 1.27 1.27)) hide)
+    )
+    (property "Datasheet" "~" (id 3) (at 142.24 135.89 0)
+      (effects (font (size 1.27 1.27)) hide)
+    )
+    (pin "1")
+  )
   (symbol (lib_id "Jumper:SolderJumper_2_Open") (at 161.29 156.21 0) (unit 1)
     (in_bom yes) (on_board yes) (fields_autoplaced)
@@
     )
     (pin "1")
+  )
+  (symbol (lib_id "Connector:TestPoint") (at 142.24 133.35 270) (unit 1)
+    (in_bom yes) (on_board yes) (fields_autoplaced)
+    (property "Reference" "TP2" (id 0) (at 147.32 132.0799 90)
+      (effects (font (size 1.27 1.27)) (justify left))
+    )
+    (property "Value" "TestPoint" (id 1) (at 147.32 134.6199 90)
+      (effects (font (size 1.27 1.27)) (justify left))
+    )
+    (property "Footprint" "TestPoint:TestPoint_Pad_D3.0mm" (id 2) (at 142.24 138.43 0)
+      (effects (font (size 1.27 1.27)) hide)
+    )
+    (property "Datasheet" "~" (id 3) (at 142.24 138.43 0)
+      (effects (font (size 1.27 1.27)) hide)
+    )
+    (pin "1")
+  )
+  (symbol (lib_id "Device:FerriteBead") (at 168.91 144.78 90) (unit 1)
+    (in_bom yes) (on_board yes) (fields_autoplaced)
+    (property "Reference" "FB1" (id 0) (at 168.8592 137.16 90))
+    (property "Value" "FerriteBead" (id 1) (at 168.8592 139.7 90))
+    (property "Footprint" "Inductor_SMD:L_0805_2012Metric_Pad1.05x1.20mm_HandSolder" (id 2) (at 168.91 146.558 90)
+      (effects (font (size 1.27 1.27)) hide)
+    )
+    (property "Datasheet" "~" (id 3) (at 168.91 144.78 0)
+      (effects (font (size 1.27 1.27)) hide)
+    )
+    (pin "1")
+    (pin "2")
   )
   (symbol (lib_id "power:GND") (at 24.13 82.55 0) (unit 1)
@@
       (reference "D6") (unit 1) (value "LED") (footprint "LED_SMD:LED_0603_1608Metric_Pad1.05x0.95mm_HandSolder")
     )
+    (path "/f250c846-829a-4be4-bab5-3cae977f2740"
+      (reference "FB1") (unit 1) (value "FerriteBead") (footprint "Inductor_SMD:L_0805_2012Metric_Pad1.05x1.20mm_HandSolder")
+    )
     (path "/b472a744-f1dd-43ec-9020-370e486042ce/10febe5f-8747-4f68-aeef-060e8a91ecdf"
       (reference "HS2_OUT1") (unit 1) (value "Conn_Coaxial") (footprint "Connector_Coaxial:SMA_Molex_73251-2120_EdgeMount_Horizontal")
@@
       (reference "SW5_2V5_OUT1") (unit 1) (value "SW_DPDT_x2") (footprint "all_lib:JS202011SCQN")
     )
+    (path "/9ed7b2f3-d5b1-42dc-95ca-de2ba1559e86"
+      (reference "TP1") (unit 1) (value "TestPoint") (footprint "TestPoint:TestPoint_Pad_D3.0mm")
+    )
+    (path "/f16964e9-cfc8-42d5-b31b-737bd3f660d0"
+      (reference "TP2") (unit 1) (value "TestPoint") (footprint "TestPoint:TestPoint_Pad_D3.0mm")
+    )
     (path "/a76b1d31-4ca3-49d9-b4c1-9ab647e9349c/0008a3a7-c6bb-454e-89fe-f5a606883615"
       (reference "TP3") (unit 1) (value "TestPoint") (footprint "TestPoint:TestPoint_Pad_D2.5mm")
@@
     )
     (path "/3f67177d-a664-4bde-aeb2-7ccc5c5d0687"
-      (reference "U1") (unit 1) (value "SC0915") (footprint "DIP-40_W15.24mm_Socket_LongPads")
+      (reference "U1") (unit 1) (value "SC0915") (footprint "all_lib:rpi_socket_fixed")
     )
     (path "/92547dd3-85e8-4996-92ae-dc1cda01b6d3"
