File: glitcher/glitcher/bifrost.kicad_sch (KiCad schematic)
At the start: 45 parts, among them J2 Conn_01x06, SW1_1V8_OUT1 SW_DPDT_x2, SW2_1V2_OUT1 SW_DPDT_x2, SW3_VADJ_OUT1 SW_DPDT_x2, SW4_3V3_OUT1 SW_DPDT_x2, SW5_2V5_OUT1 SW_DPDT_x2, U4_1V8_OUT1 LD1117S18TR_SOT223, U5_1V2_OUT1 LD1117S12TR_SOT223, U6_VADJ_OUT1 NCP1117-ADJ_SOT223, U7_3V3_OUT1 LD1117S33TR_SOT223, U8_2V5_OUT1 LD1117S25TR_SOT223

Commit message: lolsave
Parts:
- added C26, C27, C28, C29, C30, C31: C, Capacitor_SMD:C_0603_1608Metric_Pad1.08x0.95mm_HandSolder, symbol Device:C
- added L1: INDUCTOR, Inductor_SMD:L_6.3x6.3_H3, symbol pspice:INDUCTOR
- SW1_1V8_OUT1, SW2_1V2_OUT1, SW3_VADJ_OUT1, SW4_3V3_OUT1, SW5_2V5_OUT1: footprint all_lib:SW_JS202011CQN -> all_lib:JS202011SCQN
Connections:
- net GND: now also C26.2, C27.2, C28.2, C29.2, C30.2, C31.2
- new net FILT_IN: C26.1, C27.1, C28.1, L1.1
- new net FILT_OUT: C29.1, C30.1, C31.1, L1.2

Commit message: save
Parts:
- added JP4: SolderJumper_2_Open, Jumper:SolderJumper-2_P1.3mm_Open_RoundedPad1.0x1.5mm, symbol Jumper:SolderJumper_2_Open
- added TP3, TP4: TestPoint, TestPoint:TestPoint_Pad_D2.5mm, symbol Connector:TestPoint
- L1: footprint Inductor_SMD:L_6.3x6.3_H3 -> all_lib:inductor_2727_wurth
Connections:
- net FILT_IN: now also TP3.1
- net FILT_OUT: now also TP4.1
- net VCC: now also JP4.1 (A); no longer SW1_1V8_OUT1.2 (B), SW2_1V2_OUT1.2 (B), SW3_VADJ_OUT1.2 (B), SW4_3V3_OUT1.2 (B), SW5_2V5_OUT1.2 (B)
- new net VCC_SWITCHED: JP4.2 (B), SW1_1V8_OUT1.2 (B), SW2_1V2_OUT1.2 (B), SW3_VADJ_OUT1.2 (B), SW4_3V3_OUT1.2 (B), SW5_2V5_OUT1.2 (B)

Commit message: save
Connections:
- net GND: now also C14.2, C19.2
- net VCC_VADJ: now also R7.2
Changed lines of the file:
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@@
   (junction (at 142.24 156.21) (diameter 0) (color 0 0 0 0)
   )
+  (junction (at 132.08 156.21) (diameter 0) (color 0 0 0 0)
+  )
   (junction (at 68.58 77.47) (diameter 0) (color 0 0 0 0)
   )
@@
   (junction (at 140.97 92.71) (diameter 0) (color 0 0 0 0)
   )
-  (junction (at 142.24 163.83) (diameter 0) (color 0 0 0 0)
-  )
   (junction (at 68.58 60.96) (diameter 0) (color 0 0 0 0)
   )
@@
   (junction (at 160.02 26.67) (diameter 0) (color 0 0 0 0)
   )
+  (junction (at 149.86 163.83) (diameter 0) (color 0 0 0 0)
+  )
   (junction (at 100.33 26.67) (diameter 0) (color 0 0 0 0)
   )
@@
   (junction (at 62.23 140.97) (diameter 0) (color 0 0 0 0)
   )
+  (junction (at 123.19 190.5) (diameter 0) (color 0 0 0 0)
+  )
   (junction (at 63.5 156.21) (diameter 0) (color 0 0 0 0)
   )
@@
     (stroke (width 0) (type default) (color 0 0 0 0))
   )
+  (wire (pts (xy 132.08 156.21) (xy 142.24 156.21))
+    (stroke (width 0) (type default) (color 0 0 0 0))
+  )
   (wire (pts (xy 62.23 64.77) (xy 62.23 60.96))
     (stroke (width 0) (type default) (color 0 0 0 0))
@@
     (stroke (width 0) (type default) (color 0 0 0 0))
   )
+  (wire (pts (xy 132.08 156.21) (xy 132.08 165.1))
+    (stroke (width 0) (type default) (color 0 0 0 0))
+  )
   (wire (pts (xy 124.46 92.71) (xy 140.97 92.71))
     (stroke (width 0) (type default) (color 0 0 0 0))
@@
     (stroke (width 0) (type default) (color 0 0 0 0))
   )
-  (wire (pts (xy 142.24 163.83) (xy 156.21 163.83))
+  (wire (pts (xy 142.24 170.18) (xy 142.24 165.1))
+    (stroke (width 0) (type default) (color 0 0 0 0))
+  )
+  (wire (pts (xy 142.24 163.83) (xy 149.86 163.83))
     (stroke (width 0) (type default) (color 0 0 0 0))
   )
@@
     (stroke (width 0) (type default) (color 0 0 0 0))
   )
-  (wire (pts (xy 125.73 156.21) (xy 142.24 156.21))
+  (wire (pts (xy 125.73 156.21) (xy 132.08 156.21))
     (stroke (width 0) (type default) (color 0 0 0 0))
   )
@@
     (stroke (width 0) (type default) (color 0 0 0 0))
   )
+  (wire (pts (xy 149.86 190.5) (xy 123.19 190.5))
+    (stroke (width 0) (type default) (color 0 0 0 0))
+  )
   (wire (pts (xy 118.11 177.8) (xy 118.11 181.61))
     (stroke (width 0) (type default) (color 0 0 0 0))
   )
+  (wire (pts (xy 149.86 163.83) (xy 156.21 163.83))
+    (stroke (width 0) (type default) (color 0 0 0 0))
+  )
   (wire (pts (xy 124.46 170.18) (xy 118.11 170.18))
     (stroke (width 0) (type default) (color 0 0 0 0))
@@
     (stroke (width 0) (type default) (color 0 0 0 0))
   )
+  (wire (pts (xy 142.24 165.1) (xy 132.08 165.1))
+    (stroke (width 0) (type default) (color 0 0 0 0))
+  )
   (wire (pts (xy 118.11 181.61) (xy 113.03 181.61))
     (stroke (width 0) (type default) (color 0 0 0 0))
@@
     (stroke (width 0) (type default) (color 0 0 0 0))
   )
+  (wire (pts (xy 149.86 163.83) (xy 149.86 190.5))
+    (stroke (width 0) (type default) (color 0 0 0 0))
+  )
   (wire (pts (xy 121.92 36.83) (xy 100.33 36.83))
     (stroke (width 0) (type default) (color 0 0 0 0))
@@
     (stroke (width 0) (type default) (color 0 0 0 0))
   )
-  (wire (pts (xy 142.24 163.83) (xy 142.24 170.18))
-    (stroke (width 0) (type default) (color 0 0 0 0))
-  )
