File: glitcher/glitcher/glitcher.kicad_pcb (KiCad board)
At the start: 2 copper layers, 70 parts, among them J1 Barrel_Jack, J2 Conn_01x06, J3 Conn_01x03, J4 Conn_01x03, J5 Conn_01x03, J6 Conn_01x03, J7 Conn_01x03, SW1_1V8_OUT1 SW_DPDT_x2, SW2_1V2_OUT1 SW_DPDT_x2, SW3_VADJ_OUT1 SW_DPDT_x2, SW4_3V3_OUT1 SW_DPDT_x2, SW5_2V5_OUT1 SW_DPDT_x2, U1 SC0915, U2 CMOD_A7, U3 max4619cpe+, U4_1V8_OUT1 LD1117S18TR_SOT223, U5_1V2_OUT1 LD1117S12TR_SOT223, U6_VADJ_OUT1 NCP1117-ADJ_SOT223, U7_3V3_OUT1 LD1117S33TR_SOT223, U8_2V5_OUT1 LD1117S25TR_SOT223, U9_3V3ALWAYS1 LD1117S33TR_SOT223

Commit message: save
Parts:
- added ?: , , F.Cu at (246.4, 124.5)
- added ?: , , F.Cu at (246.4, 38.1)
- added D7: D_Schottky, Diode_SMD:D_SOD-123F, F.Cu at (129.5, 111.8)
- added J_LEFTEXP1: Conn_01x20, Connector_PinHeader_2.54mm:PinHeader_1x20_P2.54mm_Vertical, F.Cu at (180.3, 42.8)
- added J_LEFTEXP_OUTER1: Conn_01x20, Connector_PinHeader_2.54mm:PinHeader_1x20_P2.54mm_Vertical, F.Cu at (180.3, 38.1)
- added J_RIGHTEXP1: Conn_01x20, Connector_PinHeader_2.54mm:PinHeader_1x20_P2.54mm_Vertical, F.Cu at (180.3, 124.5)
- added J_RIGHTEXP_OUTER1: Conn_01x20, Connector_PinHeader_2.54mm:PinHeader_1x20_P2.54mm_Vertical, F.Cu at (180.3, 119.4)
- added REF**: MountingHole_2.5mm_Pad, MountingHole:MountingHole_2.5mm_Pad, F.Cu at (170.2, 38.1)
- added REF**: MountingHole_2.5mm_Pad, MountingHole:MountingHole_2.5mm_Pad, F.Cu at (91.4, 38.1)
- added REF**: MountingHole_2.5mm_Pad, MountingHole:MountingHole_2.5mm_Pad, F.Cu at (170.2, 124.5)
- added REF**: MountingHole_2.5mm_Pad, MountingHole:MountingHole_2.5mm_Pad, F.Cu at (91.4, 124.5)
- moved C14 89.1 mm to (197.2, 96.5)
- moved C18 87.3 mm to (195.5, 86.4)
- moved C11 85.3 mm to (180.3, 99.1)
- moved C12 84.0 mm to (195.5, 73.7)
- moved C8 82.5 mm to (175.2, 96.5)
- moved C19 82.4 mm to (195.5, 99.1)
- moved C16 81.3 mm to (198.1, 66.0)
- moved C13 80.4 mm to (197.2, 83.8)
- moved C3 79.6 mm to (175.2, 94.0)
- moved R7 79.4 mm to (180.3, 96.5)
- moved C15 78.3 mm to (196.1, 56.0)
- moved C21 77.9 mm to (198.1, 63.5)
- moved R6 76.6 mm to (180.3, 94.0)
- moved C5 72.5 mm to (181.1, 67.1)
- moved C2 71.0 mm to (177.8, 86.4)
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Other:
- board outline added: 165.1 x 96.5 mm
- copper layers 2 -> 4

Commit message: lolsave
Parts:
- removed ? (x2): , 
- removed the REF** at (170.2, 38.1)
- removed the REF** at (91.4, 38.1)
- removed the REF** at (170.2, 124.5)
- removed the REF** at (91.4, 124.5)
- added C26: C, Capacitor_SMD:C_0603_1608Metric_Pad1.08x0.95mm_HandSolder, F.Cu at (205.7, 105.4)
- added C27: C, Capacitor_SMD:C_0603_1608Metric_Pad1.08x0.95mm_HandSolder, F.Cu at (205.7, 100.3)
- added C28: C, Capacitor_SMD:C_0603_1608Metric_Pad1.08x0.95mm_HandSolder, F.Cu at (205.7, 102.9)
- added C29: C, Capacitor_SMD:C_0603_1608Metric_Pad1.08x0.95mm_HandSolder, F.Cu at (220.6, 102.4)
- added C30: C, Capacitor_SMD:C_0603_1608Metric_Pad1.08x0.95mm_HandSolder, F.Cu at (221.0, 104.1)
- added C31: C, Capacitor_SMD:C_0603_1608Metric_Pad1.08x0.95mm_HandSolder, F.Cu at (220.6, 100.3)
- added JP1: SolderJumper_2_Open, Jumper:SolderJumper-2_P1.3mm_Open_RoundedPad1.0x1.5mm, F.Cu at (226.1, 106.7)
- added L1: INDUCTOR, Inductor_SMD:L_6.3x6.3_H3, F.Cu at (212.1, 101.6)
- added REF**: MountingHole_2.5mm_Pad, MountingHole:MountingHole_2.5mm_Pad, F.Cu at (243.8, 118.1)
- added REF**: MountingHole_2.5mm_Pad, MountingHole:MountingHole_2.5mm_Pad, F.Cu at (243.8, 44.5)
- added REF**: MountingHole_2.5mm_Pad, MountingHole:MountingHole_2.5mm_Pad, F.Cu at (115.6, 44.5)
- added REF**: MountingHole_2.5mm_Pad, MountingHole:MountingHole_2.5mm_Pad, F.Cu at (115.6, 118.1)
- SW1_1V8_OUT1, SW2_1V2_OUT1, SW3_VADJ_OUT1, SW4_3V3_OUT1, SW5_2V5_OUT1: footprint all_lib:SW_JS202011CQN -> all_lib:JS202011SCQN
- moved J_RIGHTEXP1 93.7 mm to (231.1, 45.7), turned to -90 degrees
- moved J_LEFTEXP1 89.8 mm to (231.1, 116.8), turned to -90 degrees
- moved J_LEFTEXP_OUTER1 89.5 mm to (231.1, 111.8), turned to -90 degrees
- moved J_RIGHTEXP_OUTER1 85.3 mm to (231.1, 50.8), turned to -90 degrees
- moved U2 69.6 mm to (154.9, 109.2), turned to 180 degrees
- moved D7 68.1 mm to (160.0, 50.8), turned to -90 degrees
- moved C8 23.4 mm to (160.0, 114.3), turned to -90 degrees
- moved RV1 21.7 mm to (167.6, 114.3), turned to 180 degrees
- moved R6 20.9 mm to (175.3, 114.3), turned to 90 degrees
- moved R7 18.0 mm to (177.8, 114.3), turned to -90 degrees
- moved J1 15.2 mm to (122.8, 108.3)
- moved U1 14.2 mm to (116.8, 50.8)
- moved R8 12.1 mm to (217.5, 58.4), turned to 180 degrees
- moved D6 11.1 mm to (213.4, 58.4), turned to 0 degrees
- moved C3 10.8 mm to (182.9, 101.6)
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Connections:
- D7 pad 1: unconnected-(D7-Pad1) -> VCC
- D7 pad 2: unconnected-(D7-Pad2) -> Net-(D7-Pad2)
- J_LEFTEXP1 pad 1: unconnected-(J_LEFTEXP1-Pad1) -> GND
- J_LEFTEXP1 pad 10: unconnected-(J_LEFTEXP1-Pad10) -> RPI_GP9
- J_LEFTEXP1 pad 11: unconnected-(J_LEFTEXP1-Pad11) -> RPI_GP10
- J_LEFTEXP1 pad 12: unconnected-(J_LEFTEXP1-Pad12) -> RPI_GP11
- J_LEFTEXP1 pad 13: unconnected-(J_LEFTEXP1-Pad13) -> RPI_GP12
- J_LEFTEXP1 pad 14: unconnected-(J_LEFTEXP1-Pad14) -> RPI_GP13
- J_LEFTEXP1 pad 15: unconnected-(J_LEFTEXP1-Pad15) -> RPI_GP14
- J_LEFTEXP1 pad 16: unconnected-(J_LEFTEXP1-Pad16) -> RPI_GP15
- J_LEFTEXP1 pad 19: unconnected-(J_LEFTEXP1-Pad19) -> VCC
- J_LEFTEXP1 pad 20: unconnected-(J_LEFTEXP1-Pad20) -> GND
- J_LEFTEXP1 pad 3: unconnected-(J_LEFTEXP1-Pad3) -> RPI_GP2
- J_LEFTEXP1 pad 4: unconnected-(J_LEFTEXP1-Pad4) -> RPI_GP3
- J_LEFTEXP1 pad 5: unconnected-(J_LEFTEXP1-Pad5) -> RPI_GP4
- J_LEFTEXP1 pad 6: unconnected-(J_LEFTEXP1-Pad6) -> RPI_GP5
- J_LEFTEXP1 pad 7: unconnected-(J_LEFTEXP1-Pad7) -> RPI_GP6
- J_LEFTEXP1 pad 8: unconnected-(J_LEFTEXP1-Pad8) -> RPI_GP7
- J_LEFTEXP1 pad 9: unconnected-(J_LEFTEXP1-Pad9) -> RPI_GP8
- J_LEFTEXP_OUTER1 pad 1: unconnected-(J_LEFTEXP_OUTER1-Pad1) -> GND
- J_LEFTEXP_OUTER1 pad 10: unconnected-(J_LEFTEXP_OUTER1-Pad10) -> RPI_GP9
- J_LEFTEXP_OUTER1 pad 11: unconnected-(J_LEFTEXP_OUTER1-Pad11) -> RPI_GP10
- J_LEFTEXP_OUTER1 pad 12: unconnected-(J_LEFTEXP_OUTER1-Pad12) -> RPI_GP11
- J_LEFTEXP_OUTER1 pad 13: unconnected-(J_LEFTEXP_OUTER1-Pad13) -> RPI_GP12
- J_LEFTEXP_OUTER1 pad 14: unconnected-(J_LEFTEXP_OUTER1-Pad14) -> RPI_GP13
- J_LEFTEXP_OUTER1 pad 15: unconnected-(J_LEFTEXP_OUTER1-Pad15) -> RPI_GP14
- J_LEFTEXP_OUTER1 pad 16: unconnected-(J_LEFTEXP_OUTER1-Pad16) -> RPI_GP15
- J_LEFTEXP_OUTER1 pad 19: unconnected-(J_LEFTEXP_OUTER1-Pad19) -> VCC
- J_LEFTEXP_OUTER1 pad 20: unconnected-(J_LEFTEXP_OUTER1-Pad20) -> GND
- J_LEFTEXP_OUTER1 pad 3: unconnected-(J_LEFTEXP_OUTER1-Pad3) -> RPI_GP2
- J_LEFTEXP_OUTER1 pad 4: unconnected-(J_LEFTEXP_OUTER1-Pad4) -> RPI_GP3
- J_LEFTEXP_OUTER1 pad 5: unconnected-(J_LEFTEXP_OUTER1-Pad5) -> RPI_GP4
- J_LEFTEXP_OUTER1 pad 6: unconnected-(J_LEFTEXP_OUTER1-Pad6) -> RPI_GP5
- J_LEFTEXP_OUTER1 pad 7: unconnected-(J_LEFTEXP_OUTER1-Pad7) -> RPI_GP6
- J_LEFTEXP_OUTER1 pad 8: unconnected-(J_LEFTEXP_OUTER1-Pad8) -> RPI_GP7
- J_LEFTEXP_OUTER1 pad 9: unconnected-(J_LEFTEXP_OUTER1-Pad9) -> RPI_GP8
- J_RIGHTEXP1 pad 1: unconnected-(J_RIGHTEXP1-Pad1) -> X_OUT
- J_RIGHTEXP1 pad 10: unconnected-(J_RIGHTEXP1-Pad10) -> FPGA_GPIO_10
- J_RIGHTEXP1 pad 11: unconnected-(J_RIGHTEXP1-Pad11) -> FPGA_GPIO_9
- J_RIGHTEXP1 pad 12: unconnected-(J_RIGHTEXP1-Pad12) -> FPGA_GPIO_8
- J_RIGHTEXP1 pad 13: unconnected-(J_RIGHTEXP1-Pad13) -> FPGA_GPIO_7
- J_RIGHTEXP1 pad 14: unconnected-(J_RIGHTEXP1-Pad14) -> FPGA_GPIO_6
- J_RIGHTEXP1 pad 15: unconnected-(J_RIGHTEXP1-Pad15) -> FPGA_GPIO_5
- J_RIGHTEXP1 pad 16: unconnected-(J_RIGHTEXP1-Pad16) -> FPGA_GPIO_4
- J_RIGHTEXP1 pad 17: unconnected-(J_RIGHTEXP1-Pad17) -> FPGA_GPIO_3
- J_RIGHTEXP1 pad 18: unconnected-(J_RIGHTEXP1-Pad18) -> FPGA_GPIO_2
- J_RIGHTEXP1 pad 19: unconnected-(J_RIGHTEXP1-Pad19) -> VCC_3V3_ALWAYS
- J_RIGHTEXP1 pad 2: unconnected-(J_RIGHTEXP1-Pad2) -> Y_OUT
- J_RIGHTEXP1 pad 20: unconnected-(J_RIGHTEXP1-Pad20) -> GND
- J_RIGHTEXP1 pad 3: unconnected-(J_RIGHTEXP1-Pad3) -> Z_OUT
- J_RIGHTEXP1 pad 5: unconnected-(J_RIGHTEXP1-Pad5) -> MAX4619_A
- J_RIGHTEXP1 pad 6: unconnected-(J_RIGHTEXP1-Pad6) -> MAX4619_B
- J_RIGHTEXP1 pad 7: unconnected-(J_RIGHTEXP1-Pad7) -> MAX4619_C
- J_RIGHTEXP1 pad 8: unconnected-(J_RIGHTEXP1-Pad8) -> FPGA_GPIO_12
- J_RIGHTEXP1 pad 9: unconnected-(J_RIGHTEXP1-Pad9) -> FPGA_GPIO_11
- J_RIGHTEXP_OUTER1 pad 1: unconnected-(J_RIGHTEXP_OUTER1-Pad1) -> X_OUT
- J_RIGHTEXP_OUTER1 pad 10: unconnected-(J_RIGHTEXP_OUTER1-Pad10) -> FPGA_GPIO_10
- J_RIGHTEXP_OUTER1 pad 11: unconnected-(J_RIGHTEXP_OUTER1-Pad11) -> FPGA_GPIO_9
- J_RIGHTEXP_OUTER1 pad 12: unconnected-(J_RIGHTEXP_OUTER1-Pad12) -> FPGA_GPIO_8
- J_RIGHTEXP_OUTER1 pad 13: unconnected-(J_RIGHTEXP_OUTER1-Pad13) -> FPGA_GPIO_7
- J_RIGHTEXP_OUTER1 pad 14: unconnected-(J_RIGHTEXP_OUTER1-Pad14) -> FPGA_GPIO_6
- J_RIGHTEXP_OUTER1 pad 15: unconnected-(J_RIGHTEXP_OUTER1-Pad15) -> FPGA_GPIO_5
- J_RIGHTEXP_OUTER1 pad 16: unconnected-(J_RIGHTEXP_OUTER1-Pad16) -> FPGA_GPIO_4
- J_RIGHTEXP_OUTER1 pad 17: unconnected-(J_RIGHTEXP_OUTER1-Pad17) -> FPGA_GPIO_3
- J_RIGHTEXP_OUTER1 pad 18: unconnected-(J_RIGHTEXP_OUTER1-Pad18) -> FPGA_GPIO_2
- J_RIGHTEXP_OUTER1 pad 19: unconnected-(J_RIGHTEXP_OUTER1-Pad19) -> VCC_3V3_ALWAYS
- J_RIGHTEXP_OUTER1 pad 2: unconnected-(J_RIGHTEXP_OUTER1-Pad2) -> Y_OUT
- J_RIGHTEXP_OUTER1 pad 20: unconnected-(J_RIGHTEXP_OUTER1-Pad20) -> GND
- J_RIGHTEXP_OUTER1 pad 3: unconnected-(J_RIGHTEXP_OUTER1-Pad3) -> Z_OUT
- J_RIGHTEXP_OUTER1 pad 5: unconnected-(J_RIGHTEXP_OUTER1-Pad5) -> MAX4619_A
- J_RIGHTEXP_OUTER1 pad 6: unconnected-(J_RIGHTEXP_OUTER1-Pad6) -> MAX4619_B
- J_RIGHTEXP_OUTER1 pad 7: unconnected-(J_RIGHTEXP_OUTER1-Pad7) -> MAX4619_C
- J_RIGHTEXP_OUTER1 pad 8: unconnected-(J_RIGHTEXP_OUTER1-Pad8) -> FPGA_GPIO_12
- J_RIGHTEXP_OUTER1 pad 9: unconnected-(J_RIGHTEXP_OUTER1-Pad9) -> FPGA_GPIO_11
- R8 pad 1: VCC -> VCC_3V3_ALWAYS
- U1 pad 1: unconnected-(U1-Pad1) -> RPI_GP0
- U1 pad 10: unconnected-(U1-Pad10) -> RPI_GP7
- U1 pad 11: unconnected-(U1-Pad11) -> RPI_GP8
- U1 pad 12: unconnected-(U1-Pad12) -> RPI_GP9
- U1 pad 14: unconnected-(U1-Pad14) -> RPI_GP10
- U1 pad 15: unconnected-(U1-Pad15) -> RPI_GP11
- U1 pad 16: unconnected-(U1-Pad16) -> RPI_GP12
- U1 pad 17: unconnected-(U1-Pad17) -> RPI_GP13
- U1 pad 19: unconnected-(U1-Pad19) -> RPI_GP14
- U1 pad 2: unconnected-(U1-Pad2) -> RPI_GP1
- U1 pad 20: unconnected-(U1-Pad20) -> RPI_GP15
- U1 pad 21: unconnected-(U1-Pad21) -> RPI_GP16
- U1 pad 22: unconnected-(U1-Pad22) -> RPI_GP17
- U1 pad 4: unconnected-(U1-Pad4) -> RPI_GP2
- U1 pad 5: unconnected-(U1-Pad5) -> RPI_GP3
- U1 pad 6: unconnected-(U1-Pad6) -> RPI_GP4
- U1 pad 7: unconnected-(U1-Pad7) -> RPI_GP5
- U1 pad 9: unconnected-(U1-Pad9) -> RPI_GP6
- U2 pad 1: unconnected-(U2-Pad1) -> MAX4619_C
- U2 pad 10: unconnected-(U2-Pad10) -> FPGA_GPIO_6
- U2 pad 11: unconnected-(U2-Pad11) -> FPGA_GPIO_5
- U2 pad 12: unconnected-(U2-Pad12) -> FPGA_GPIO_4
- U2 pad 13: unconnected-(U2-Pad13) -> FPGA_GPIO_3
- U2 pad 14: unconnected-(U2-Pad14) -> FPGA_GPIO_2
- U2 pad 15: unconnected-(U2-Pad15) -> FPGA_GPIO_1
- U2 pad 2: unconnected-(U2-Pad2) -> MAX4619_B
- U2 pad 24: VCC -> Net-(D7-Pad2)
- U2 pad 26: unconnected-(U2-Pad26) -> RPI_GP0
- U2 pad 27: unconnected-(U2-Pad27) -> RPI_GP1
- U2 pad 3: unconnected-(U2-Pad3) -> MAX4619_A
- U2 pad 4: unconnected-(U2-Pad4) -> FPGA_GPIO_12
- U2 pad 5: unconnected-(U2-Pad5) -> FPGA_GPIO_11
- U2 pad 6: unconnected-(U2-Pad6) -> FPGA_GPIO_10
- U2 pad 7: unconnected-(U2-Pad7) -> FPGA_GPIO_9
- U2 pad 8: unconnected-(U2-Pad8) -> FPGA_GPIO_8
- U2 pad 9: unconnected-(U2-Pad9) -> FPGA_GPIO_7
Routing:
- net GND: track 0.00 -> 871.1 mm, vias 0 -> 15
- net VCC: track 0.00 -> 361.6 mm, vias 0 -> 8
- net RPI_GP2: track 0.00 -> 140.8 mm
- net RPI_GP3: track 0.00 -> 132.8 mm
- net MAX4619_C: track 0.00 -> 131.3 mm
- net RPI_GP4: track 0.00 -> 130.3 mm
- net RPI_GP5: track 0.00 -> 127.8 mm
- net MAX4619_B: track 0.00 -> 127.7 mm
- net MAX4619_A: track 0.00 -> 124.3 mm
- net RPI_GP6: track 0.00 -> 121.0 mm
- net RPI_GP7: track 0.00 -> 117.4 mm
- net RPI_GP8: track 0.00 -> 114.9 mm
- net RPI_GP9: track 0.00 -> 110.2 mm
- net RPI_GP10: track 0.00 -> 105.6 mm
- net RPI_GP11: track 0.00 -> 102.0 mm
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Other:
- board size 165.1 x 96.5 mm -> 135.9 x 81.3 mm

Commit message: save
Parts:
- removed D7: D_Schottky, Diode_SMD:D_SOD-123F
- added JP2: SolderJumper_2_Open, Jumper:SolderJumper-2_P1.3mm_Open_Pad1.0x1.5mm, F.Cu at (130.2, 45.7)
- added JP3: SolderJumper_2_Open, Jumper:SolderJumper-2_P1.3mm_Open_Pad1.0x1.5mm, F.Cu at (153.1, 45.7)
- added JP4: SolderJumper_2_Open, Jumper:SolderJumper-2_P1.3mm_Open_RoundedPad1.0x1.5mm, F.Cu at (145.5, 113.0)
- added R10: 10K R, Resistor_SMD:R_0603_1608Metric_Pad0.98x0.95mm_HandSolder, F.Cu at (230.6, 101.6)
- added R9: 1R, Resistor_SMD:R_0603_1608Metric_Pad0.98x0.95mm_HandSolder, F.Cu at (230.6, 104.1)
- added REF**: TestPoint_Plated_Hole_D2.0mm, TestPoint:TestPoint_Plated_Hole_D2.0mm, F.Cu at (230.6, 107.3)
- added TP3: TestPoint, TestPoint:TestPoint_Pad_D2.5mm, F.Cu at (205.2, 96.5)
- added TP4: TestPoint, TestPoint:TestPoint_Pad_D2.5mm, F.Cu at (217.9, 96.5)
- added U4: irf7807z, Package_SO:SOIC-8-1EP_3.9x4.9mm_P1.27mm_EP2.29x3mm, F.Cu at (230.6, 96.5)
- L1: footprint Inductor_SMD:L_6.3x6.3_H3 -> all_lib:inductor_2727_wurth
- moved C30 3.35 mm to (217.9, 105.4)
- moved C29 2.73 mm to (217.9, 102.9)
- moved C31 2.69 mm to (217.9, 100.3)
- moved L1 2.48 mm to (212.8, 99.2)
- moved C24 0.58 mm to (233.1, 63.5)
- moved C26 0.58 mm to (205.2, 105.4)
- moved C27 0.58 mm to (205.2, 100.3)
- moved C28 0.58 mm to (205.2, 102.9)
- moved C8 0.58 mm to (159.4, 114.3)
- moved D6 0.58 mm to (212.8, 58.4)
- moved HS2_OUT1 0.58 mm to (245.3, 94.0)
- moved J3 0.58 mm to (237.7, 91.4)
- moved J4 0.58 mm to (237.7, 53.3)
- moved J5 0.58 mm to (237.7, 66.0)
- moved J6 0.58 mm to (237.7, 104.1)
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Connections:
- C22 pad 1: VCC -> VCC_SWITCHED
- C23 pad 1: VCC -> VCC_SWITCHED
- J_LEFTEXP1 pad 17: unconnected-(J_LEFTEXP1-Pad17) -> FREE_LEFT17
- J_LEFTEXP1 pad 18: unconnected-(J_LEFTEXP1-Pad18) -> FREE_LEFT18
- J_LEFTEXP1 pad 19: VCC -> VCC_SWITCHED
- J_LEFTEXP1 pad 2: unconnected-(J_LEFTEXP1-Pad2) -> FREE_LEFT2
- J_LEFTEXP_OUTER1 pad 17: unconnected-(J_LEFTEXP_OUTER1-Pad17) -> FREE_LEFT17
- J_LEFTEXP_OUTER1 pad 18: unconnected-(J_LEFTEXP_OUTER1-Pad18) -> FREE_LEFT18
- J_LEFTEXP_OUTER1 pad 19: VCC -> VCC_SWITCHED
- J_LEFTEXP_OUTER1 pad 2: unconnected-(J_LEFTEXP_OUTER1-Pad2) -> FREE_LEFT2
- J_RIGHTEXP1 pad 4: unconnected-(J_RIGHTEXP1-Pad4) -> FREE_RIGHT4
- J_RIGHTEXP_OUTER1 pad 4: unconnected-(J_RIGHTEXP_OUTER1-Pad4) -> FREE_RIGHT4
- SW1_1V8_OUT1 pad 2: VCC -> VCC_SWITCHED
- SW2_1V2_OUT1 pad 2: VCC -> VCC_SWITCHED
- SW3_VADJ_OUT1 pad 2: VCC -> VCC_SWITCHED
- SW4_3V3_OUT1 pad 2: VCC -> VCC_SWITCHED
- SW5_2V5_OUT1 pad 2: VCC -> VCC_SWITCHED
- U1 pad 39: VCC -> Net-(JP2-Pad1)
- U9_3V3ALWAYS1 pad 3: VCC -> VCC_SWITCHED
Routing:
- net VCC_SWITCHED: track 0.00 -> 204.4 mm, vias 0 -> 7
- net VCC: track 361.6 -> 160.9 mm, vias 8 -> 1
- net GND: track 871.1 -> 946.6 mm, vias 15 -> 16
- net FILT_IN: track 0.00 -> 24.0 mm
- net FILT_OUT: track 0.00 -> 14.5 mm
- net Net-(JP2-Pad1): track 0.00 -> 9.14 mm
- net HS2_OUT: track 7.49 -> 16.3 mm
- net Net-(R10-Pad1): track 0.00 -> 7.24 mm
- net RPI_GP0: track 23.9 -> 29.8 mm
- net FREE_RIGHT4: track 0.00 -> 5.08 mm
- net FREE_LEFT2: track 0.00 -> 5.08 mm
- net FREE_LEFT18: track 0.00 -> 5.08 mm
- net FREE_LEFT17: track 0.00 -> 5.08 mm
- net GL_GATE: track 0.00 -> 3.55 mm
- net Net-(D6-Pad2): track 0.00 -> 2.38 mm
Other:
- board text added: "3.3V"
- board text added: "5V"
- board text added: "FREE"
- board text added: "GL_OUT"
- board text added: "GND"
- board text added: "GND / GL_GATE"
- board text added: "GND 3.3v 2.5v 1.8v 1.2v VADJ"
- board text added: "GP10"
- board text added: "GP11"
- board text added: "GP12"
- board text added: "GP13"
- board text added: "GP14"
- board text added: "GP15"
- board text added: "GP2 / EN"
- board text added: "GP3"
- board text added: "GP4"
- board text added: "GP5"
- board text added: "GP6"
- board text added: "GP7"
- board text added: "GP8"
- board text added: "GP9"
- board text added: "MAX4619A"
- board text added: "MAX4619B"
- board text added: "MAX4619C"
- board text added: "PIO10 / J3"
- board text added: "PIO11 / J1"
- board text added: "PIO12 / K2"
- board text added: "PIO13 / L1"
- board text added: "PIO14 / L2"
- board text added: "PIO4 / K3"
- board text added: "PIO5 / C15"
- board text added: "PIO6 / H1"
- board text added: "PIO7 / A15"
- board text added: "PIO8 / B15"
- board text added: "PIO9 / A14"
- board text added: "SPARE"
- board text added: "X OUT"
- board text added: "X1 X0"
- board text added: "X_OUT"
- board text added: "Y OUT"
- board text added: "Y1 Y0"
- board text added: "Y_OUT"
- board text added: "Z1 Z0"
- board text added: "Z_OUT"

Commit message: prod1
Parts:
- added FB1: FerriteBead, Inductor_SMD:L_0805_2012Metric_Pad1.05x1.20mm_HandSolder, F.Cu at (137.7, 45.7)
- added TP1: TestPoint, TestPoint:TestPoint_Pad_D3.0mm, B.Cu at (101.6, 59.7)
- added TP2: TestPoint, TestPoint:TestPoint_Pad_D3.0mm, B.Cu at (101.6, 66.0)
- U1: footprint Package_DIP:DIP-40_W15.24mm_Socket_LongPads -> all_lib:rpi_socket_fixed
- moved REF** 24.9 mm to (90.1, 118.1)
- moved J1 24.9 mm to (97.4, 108.3)
- moved REF** 24.8 mm to (90.2, 44.5)
- moved U1 23.6 mm to (92.7, 50.8)
- moved C1 19.8 mm to (162.5, 83.8)
- moved C10 19.8 mm to (162.5, 71.1)
- moved C11 19.8 mm to (162.5, 104.1)
- moved C12 19.8 mm to (177.7, 78.7)
- moved C13 19.8 mm to (177.7, 88.9)
- moved C14 19.8 mm to (177.7, 99.1)
- moved C15 19.8 mm to (177.7, 61.1)
- moved C16 19.8 mm to (177.7, 71.1)
- moved C17 19.8 mm to (177.7, 81.3)
- moved C18 19.8 mm to (177.7, 91.4)
- moved C19 19.8 mm to (177.7, 101.6)
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Connections:
- U1 pad 27: unconnected-(U1-Pad27) -> FPGA_4
- U1 pad 29: unconnected-(U1-Pad29) -> FPGA_3
- U1 pad 31: unconnected-(U1-Pad31) -> Net-(TP2-Pad1)
- U1 pad 32: unconnected-(U1-Pad32) -> Net-(TP1-Pad1)
- U2 pad 28: unconnected-(U2-Pad28) -> FPGA_3
- U2 pad 29: unconnected-(U2-Pad29) -> FPGA_4
Routing:
- net FPGA_4: track 0.00 -> 26.0 mm
- net FPGA_3: track 0.00 -> 23.5 mm
- net VCC: track 160.9 -> 178.6 mm
- net Net-(TP1-Pad1): track 0.00 -> 15.1 mm
- net Net-(TP2-Pad1): track 0.00 -> 12.0 mm
- net GND: track 946.6 -> 954.4 mm
- net RPI_GP0: track 29.8 -> 36.7 mm
- net Net-(FB1-Pad2): track 5.34 -> 12.2 mm
- net RPI_GP2: track 140.8 -> 146.8 mm
- net RPI_GP1: track 23.9 -> 28.9 mm
- net RPI_GP7: track 117.4 -> 122.1 mm, vias 0 -> 1
- net RPI_GP14: track 90.1 -> 93.9 mm
- net RPI_GP11: track 102.0 -> 105.7 mm
- net RPI_GP15: track 86.5 -> 90.3 mm
- net RPI_GP6: track 121.0 -> 124.7 mm
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Other:
- board size 135.9 x 81.3 mm -> 140.8 x 81.3 mm
- board text added: "ADC0"
- board text added: "ADC1"
- board text added: "F"
- board text added: "GP2/ EN"
- board text added: "MAX4619A:A16"
- board text added: "MAX4619B:L3"
- board text added: "MAX4619C:M3"
- board text added: "PIO04:K3"
- board text added: "PIO05:C15"
- board text added: "PIO06:H1"
- board text added: "PIO07:A15"
- board text added: "PIO08:B15"
- board text added: "PIO09:A14"
- board text added: "PIO10:J3"
- board text added: "PIO11:J1"
- board text added: "PIO12:K2"
- board text added: "PIO13:L1"
- board text added: "PIO14:L2"
- board text added: "X"
- board text added: "Y"
- board text added: "Z"
- board text removed: "GND / GL_GATE"
- board text removed: "GP2 / EN"
- board text removed: "MAX4619A"
- board text removed: "MAX4619B"
- board text removed: "MAX4619C"
- board text removed: "PIO10 / J3"
- board text removed: "PIO11 / J1"
- board text removed: "PIO12 / K2"
- board text removed: "PIO13 / L1"
- board text removed: "PIO14 / L2"
- board text removed: "PIO4 / K3"
- board text removed: "PIO5 / C15"
- board text removed: "PIO6 / H1"
- board text removed: "PIO7 / A15"
- board text removed: "PIO8 / B15"
- board text removed: "PIO9 / A14"
- board text removed: "X_OUT"
- board text removed: "Y_OUT"

Commit message: save
Connections:
- C14 pad 2: Net-(C14-Pad2) -> GND
- C19 pad 2: Net-(C14-Pad2) -> GND
- R7 pad 2: Net-(C14-Pad2) -> VCC_VADJ
Routing:
- net Net-(C14-Pad2): track 29.4 -> 0.00 mm
- net VCC_VADJ: track 38.5 -> 63.9 mm
- net GND: track 954.4 -> 968.9 mm, vias 16 -> 17
